File: eagle/hwep_sequencer_v2/Beilage.brd (EAGLE design)
At the start: 251.5 x 94 mm, 142 parts, among them X1 ESP32-DEVKIT-C

Commit message: Prescaler Sim
Optimised Schematic
Changed unavailable ICs
Issue: Interrupt on Input MCP23S08 and Prescaler Strobe
Parts:
- removed R31, R33: 10k, rcl_GruS:R0805
- removed R32, R34: 2k7, rcl_GruS:R0805
- added C31: 100n, rcl_GruS:C0805
- added R14: 10k, rcl_GruS:R0805
- added R18: 100R, rcl_GruS:R0805
- added R2, R9: 10k, rcl_GruS:P160LB
- added X3, X4: (no value), con_GruS:MYLIB_SJ
- C10, C25, C29: value 100n -> 1u
- C23, C27, C8: value 1u -> 100n
- C4: value 10n -> 4u7
- C6: value 100n -> 10n
- D11, D13: value 74AHC1G04DBV -> 74AHC1G125DBV
- D9: value 74AHCT1G125DBV -> 74AHC1G125DBV
- R12, R13: device rcl_GruS:P160LB -> rcl_GruS:R0805
- R16, R17, R19: value 10k -> 100R
- R24, R25, R26: value 100R -> 100k
- R27: value 100R -> 10k
- R28, R30: value 100k -> 2k7
- R29: value 100k -> 10k
- R6: value 10k -> 1k; device rcl_GruS:P160LB -> rcl_GruS:R0805
- R8: value 1k -> 10k; device rcl_GruS:R0805 -> rcl_GruS:P160LB
- S14: value EC11E09244AQ -> (none); device switch_GruS:EC11 -> switch_GruS:B3F-10XX
- S15: value (none) -> EC11E09244AQ; device switch_GruS:B3F-10XX -> switch_GruS:EC11
- moved R8 226.5 mm to (11.4, 11.4), turned to 0 degrees
- moved C27 171.8 mm to (212.1, 80.0), turned to 0 degrees
- moved C29 125.6 mm to (42.5, 40.6)
- moved R6 123.7 mm to (172.7, 83.8), turned to 270 degrees
- moved C10 108.4 mm to (105.4, 58.4), turned to 180 degrees
- moved R12 107.6 mm to (238.8, 33.0), turned to 90 degrees
- moved R3 101.6 mm to (113.0, 11.4)
- moved R4 101.6 mm to (133.3, 11.4)
- moved R5 101.6 mm to (153.7, 11.4)
- moved R13 90.3 mm to (241.3, 33.0), turned to 90 degrees
- moved S14 89.1 mm to (133.3, 83.8), turned to 270 degrees
- moved S15 89.1 mm to (191.8, 16.5), turned to 0 degrees
- moved C8 89.1 mm to (172.1, 17.1), turned to 270 degrees
- moved R15 73.3 mm to (166.4, 21.6), turned to 0 degrees
- moved C23 69.3 mm to (242.6, 17.8)
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Connections:
- removed net N$1: D6.15, D7.5
- new net INT_23S08: D1.8
- new net PSGS: D8.11
- net +3V3: now also C10.1, C31.1, D11.2, D13.2, R12.2, R13.2, R14.2; no longer C23.1, C7.1, R16.2, R17.2, R19.2, R31.2, R33.2
- net +5V: now also C23.1, X4.1; no longer C10.1
- net 088S052_!CS!: now also R15.1; no longer R19.1
- net 7SEG_A: now also R23.2; no longer R27.2
- net 7SEG_B: now also R22.2; no longer R26.2
- net 7SEG_C: now also R21.2; no longer R25.2
- net 7SEG_CE: now also R24.2; no longer R28.2
- net 7SEG_CH: now also R26.2; no longer R30.2
- net 7SEG_CZ: now also R25.2; no longer R29.2
- net 7SEG_D: now also R20.2; no longer R24.2
- net 7SEG_DP: now also R16.2; no longer R20.2
- net 7SEG_E: now also R19.2; no longer R23.2
- net 7SEG_F: now also R18.2; no longer R22.2
- net 7SEG_G: now also R17.2; no longer R21.2
- net ADC0: now also R8.2; no longer R3.2
- net ADC1: now also R9.2; no longer R4.2
- net ADC2: now also R10.2; no longer R5.2
- net ADC3: now also R11.2; no longer R6.2
- net ADC4: now also R2.2; no longer R10.2
- net ADC5: now also R3.2; no longer R11.2
- net ADC6: now also R4.2; no longer R12.2
- net ADC7: now also R5.2; no longer R13.2
- net AGND: now also C4.2, C7.2, R10.3, R11.3, R2.3, R3.3, R4.3, R5.3, R8.3, R9.3, X3.2; no longer C6.2, R10.1, R11.1, R12.1, R13.1, R3.1, R4.1, R5.1, R6.1
- net EC11_A: now also C5.1, R12.1, S15.A1; no longer C4.1, R15.1, S14.A1
- net EC11_B: now also C6.1, R13.1, S15.B1; no longer C5.1, R16.1, S14.B1
- net EC11_SW: now also R14.1, S15.E1; no longer R17.1, S14.E1
- net GND: now also C31.2, C6.2, R24.1, R25.1, R26.1, R27.1, R6.1, S14.1, S14.2, S15.C1, S15.D1, S15.MH1, S15.MH2, X3.1; no longer C4.2, C7.2, R32.1, R34.1, R8.1, S14.C1, S14.D1, S14.MH1, S14.MH2, S15.1, S15.2
- net N$24: now also R28.2; no longer R32.2
- net N$33: now also R17.1; no longer R21.1
- net N$35: now also R18.1; no longer R22.1
- net N$36: now also R23.1; no longer R27.1
- net N$37: now also R22.1; no longer R26.1
- net N$54: now also R30.2; no longer R34.2
- net N$56: now also R20.1; no longer R24.1
- net N$58: now also R6.2; no longer R7.2
- net N$61: now also R29.2; no longer R33.1
- net N$66: now also R27.2; no longer R31.1
- net N$7: now also R16.1; no longer R20.1
- net N$78: now also R21.1; no longer R25.1
- net N$80: now also R19.1; no longer R23.1
- net N$9: now also R7.2; no longer R8.2
- net PS3: now also D6.15, D7.5; no longer D8.11
- net RESET_CNT: now also S14.3; no longer S15.3
- net STP_LE_K: now also D11.1; no longer D11.2
- net STP_LE_S: now also D13.1; no longer D13.2
- net VREF: now also C4.1, C7.1, R10.1, R11.1, R2.1, R3.1, R4.1, R5.1, R8.1, R9.1, X4.2; no longer C6.1, R10.3, R11.3, R12.3, R13.3, R3.3, R4.3, R5.3, R6.3
Routing:
- net VREF: track 187.8 -> 286.5 mm, vias 1 -> 2
- net AGND: track 197.1 -> 276.2 mm
- net PS3: track 25.4 -> 70.8 mm
- net +3V3: track 879.4 -> 854.1 mm, vias 8 -> 7
- net N$1: track 13.3 -> 0.00 mm
- net +5V: track 205.2 -> 210.1 mm
- net N$61: track 9.19 -> 14.0 mm
- net PS_G0: track 42.9 -> 47.4 mm
- net N$66: track 15.9 -> 19.4 mm, vias 1 -> 2
- net INT_23S08: track 0.00 -> 2.14 mm, vias 0 -> 1
- net N$9: track 2.87 -> 4.14 mm
- net STP_LE_S: track 43.5 -> 44.6 mm
- net STP_LE_K: track 12.8 -> 13.9 mm, vias 0 -> 1
