File: eagle/hwep_sequencer_v2/Beilage.brd (EAGLE design)
At the start: 227.3 x 82.5 mm, 119 parts, among them X1 ESP32CLIP2122

Commit message: updated outline
Parts:
- removed FABRICATION: (no value), fabrication:FABRIACTION
- added R27, R28, R31, R32, R33, R34, R35, R36, R37, R38: 18k, rcl_GruS:R0805
- moved R29 15.5 mm to (184.2, 45.7)
- moved C10 8.52 mm to (101.6, 55.9), turned to 90 degrees
- moved C9 5.68 mm to (100.3, 68.6), turned to 90 degrees
Connections:
- net DI renamed N$1
- net DO renamed N$2
- net +3V3: now also R27.2, R28.2, R31.2, R32.2, R33.2, R34.2, R35.2, R36.2, R37.2, R38.2
- net EVENT: now also S12.3; no longer S12.4
- net MOSI: now also D1.2, D5.14
- net PSGS: now also X1.7
- net Q0_SW_BD: now also R28.1
- net Q0_SW_GD: now also R35.1
- net Q1_SW_BD: now also R31.1
- net Q1_SW_GD: now also R36.1
- net Q2_SW_BD: now also R32.1
- net Q2_SW_GD: now also R37.1
- net Q3_SW_BD: now also R33.1
- net Q3_SW_GD: now also R38.1
- net SRC_SW_BD: now also R27.1
- net SRC_SW_GD: now also R34.1
Routing:
- net PSGS: track 0.00 -> 58.8 mm, vias 0 -> 1
- net +3V3: track 678.4 -> 729.4 mm
- net MOSI: track 38.3 -> 72.6 mm
- net ADC088S052_!CS: track 93.1 -> 80.5 mm, vias 1 -> 3
- net Q2_SW_GD: track 56.2 -> 65.3 mm, vias 1 -> 2
- net Q3_SW_GD: track 28.3 -> 35.8 mm
- net Q2_SW_BD: track 54.1 -> 61.2 mm
- net SRC_SW_BD: track 108.1 -> 113.5 mm, vias 0 -> 1
- net Q1_SW_GD: track 72.5 -> 77.9 mm, vias 0 -> 1
- net N$55: track 23.9 -> 19.5 mm
- net Q0_SW_GD: track 90.3 -> 94.4 mm, vias 0 -> 1
- net Q0_SW_BD: track 90.3 -> 94.4 mm, vias 0 -> 1
- net EVENT: track 19.4 -> 15.7 mm
- net PS_G0: track 47.4 -> 51.0 mm
- net Q3_SW_BD: track 26.2 -> 29.4 mm
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
Commit message: Finalised Board
Parts:
- added FABRICATION: (no value), fabrication:FABRIACTION
- R27, R28, R31, R32, R33, R34, R35, R36, R37, R38: value 18k -> 47k
- moved C28 15.2 mm to (27.3, 41.9), flipped to the bottom, turned to 0 degrees
- moved C29 15.2 mm to (27.3, 30.5), flipped to the bottom, turned to 0 degrees
Routing:
- net AGND: track 302.2 -> 106.7 mm, vias 2 -> 1
- net +3V3: track 729.4 -> 719.2 mm
- net GND: vias 14 -> 15
- added copper zone on layer 1, net AGND
- added copper zone on layer 16, net AGND

Commit message: finale gerber generation
Parts:
- removed C28: 1u, rcl_GruS:C0805
- removed D12: STP16CP05TTR, ic_GruS:TSSOP24
- removed R33, R34, R35, R36, R37, R38: 47k, rcl_GruS:R0805
- added C2: 1u, rcl_GruS:C0805
- added D4: ADC088S052, adc-dac_GruS:TSSOP16
- C10: value 1u -> 100n
- C23, C8: value 100n -> 1u
- C3: value 1u -> 10n
- C4: value 4u7 -> 10n
- C5, C6: value 10n -> 100n
- C7: value 100n -> 4u7
- D5: value ADC088S052 -> 74HC148N; device adc-dac_GruS:TSSOP16 -> 74xx_GruS:DIP16
- D7: value 74HC148N -> 74HC00N; device 74xx_GruS:DIP16 -> 74xx_GruS:DIP14
- D8: value 74HC00N -> 74AHC1G125DBV; device 74xx_GruS:DIP14 -> 74xx_GruS:SOT23-5
- D9: value 74AHC1G125DBV -> STP16CP05TTR; device 74xx_GruS:SOT23-5 -> ic_GruS:TSSOP24
- R1: device rcl_GruS:R0805 -> rcl_GruS:P160LB
- R10, R9: value 10k -> 1k; device rcl_GruS:P160LB -> rcl_GruS:R0805
- R11: value 10k -> 47k; device rcl_GruS:P160LB -> rcl_GruS:R0805
- R12, R13, R14, R15: value 10k -> 47k
- R16, R17, R18, R19, R20: value 100R -> 47k
- R24, R25, R26: value 100k -> 100R
- R27, R28: value 47k -> 100R
- R29: value 10k -> 100k
- R30: value 2k7 -> 100k
- R31: value 47k -> 100k
- R32: value 47k -> 2k7
- R6, R7: value 1k -> 10k; device rcl_GruS:R0805 -> rcl_GruS:P160LB
- S11: value (none) -> EC11E09244AQ; device switch_GruS:B3F-10XX -> switch_GruS:EC11
- S15: value EC11E09244AQ -> (none); device switch_GruS:EC11 -> switch_GruS:B3F-10XX
- moved C23 192.4 mm to (27.3, 41.9), flipped to the bottom, turned to 0 degrees
- moved R1 148.6 mm to (11.4, 24.1), flipped to the top, turned to 180 degrees
- moved R8 142.2 mm to (153.7, 24.1)
- moved R9 140.8 mm to (162.6, 76.2), turned to 0 degrees
- moved R10 127.9 mm to (168.9, 76.2)
- moved R14 124.9 mm to (77.5, 68.6), turned to 270 degrees
- moved R12 124.9 mm to (82.5, 68.6), turned to 270 degrees
- moved R13 124.9 mm to (80.0, 68.6), turned to 270 degrees
- moved R15 120.3 mm to (87.6, 68.6), turned to 270 degrees
- moved C10 115.3 mm to (212.1, 22.9)
- moved R31 114.8 mm to (194.3, 78.7), flipped to the bottom
- moved R16 96.6 mm to (80.0, 61.0), flipped to the top, turned to 90 degrees
- moved R19 94.8 mm to (77.5, 61.0), flipped to the top, turned to 90 degrees
- moved R27 91.5 mm to (176.5, 66.0), flipped to the bottom, turned to 0 degrees
- moved R18 91.4 mm to (85.1, 61.0), flipped to the top, turned to 90 degrees
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- renumbered C29 to C24, C30 to C25, H34 to H18, H35 to H19, H36 to H20, H37 to H21, H38 to H22, H39 to H23, H40 to H24, H41 to H25, H42 to H26, H43 to H27, H44 to H28, H45 to H29, H46 to H30, H47 to H31, H48 to H32, H49 to H33
Connections:
- removed net N$2 (its old number): H14.2, H3.4
- new net N$4: H11.4, H8.2
- net +3V3: now also C2.1, C23.1, C6.1, D4.13, D5.10, D5.11, D5.12, D5.16, D7.14, D9.24, R11.2, R16.2, R17.2, R18.2, R19.2, R20.2; no longer C10.1, C28.1, C3.1, D12.24, D5.13, D7.10, D7.11, D7.12, D7.16, D8.14, R1.2, R27.2, R28.2, R31.2, R32.2, R33.2, R34.2, R35.2, R36.2, R37.2, R38.2
- net +5V: now also C10.1, D8.5; no longer C23.1, D9.5
- net 23S08_!CS: no longer R1.1
- net 7SEG_A: now also R28.2; no longer R23.2
- net 7SEG_B: now also R27.2; no longer R22.2
- net 7SEG_C: now also R26.2; no longer R21.2
- net 7SEG_CE: now also R29.2; no longer R24.2
- net 7SEG_CH: now also R31.2; no longer R26.2
- net 7SEG_CZ: now also R30.2; no longer R25.2
- net 7SEG_D: now also R25.2; no longer R20.2
- net 7SEG_DP: now also R21.2; no longer R16.2
- net 7SEG_E: now also R24.2; no longer R19.2
- net 7SEG_F: now also R23.2; no longer R18.2
- net 7SEG_G: now also R22.2; no longer R17.2
- net ADC0: now also D4.4, R1.2; no longer D5.4, R8.2
- net ADC088S052_!CS: now also D4.1; no longer D5.1, R15.1
- net ADC1: now also D4.5, R2.2; no longer D5.5, R9.2
- net ADC2: now also D4.6, R3.2; no longer D5.6, R10.2
- net ADC3: now also D4.7, R4.2; no longer D5.7, R11.2
- net ADC4: now also D4.8, R5.2; no longer D5.8, R2.2
- net ADC5: now also D4.9, R6.2; no longer D5.9, R3.2
- net ADC6: now also D4.10, R7.2; no longer D5.10, R4.2
- net ADC7: now also D4.11, R8.2; no longer D5.11, R5.2
- net AGND: now also C5.2, D4.3, R1.3, R6.3, R7.3; no longer C4.2, D5.3, R10.3, R11.3, R9.3
- net EC11_A: now also C3.1, S11.A1; no longer C5.1, R12.1, S15.A1
- net EC11_B: now also C4.1, S11.B1; no longer C6.1, R13.1, S15.B1
- net EC11_SW: now also S11.E1; no longer R14.1, S15.E1
- net EVENT: now also S13.3; no longer S12.3
- net GND: now also C2.2, C4.2, D4.12, D5.5, D5.8, D7.7, D8.1, D8.3, D9.21, R10.1, R31.1, R32.1, R9.1, S11.C1, S11.D1, S11.MH1, S11.MH2, S15.1, S15.2; no longer C28.2, C5.2, D12.1, D12.21, D5.12, D6.5, D7.8, D8.7, D9.3, R24.1, R25.1, R26.1, R6.1, R7.1, S11.1, S11.2, S15.C1, S15.D1, S15.MH1, S15.MH2
- net GS_B: now also D5.14, D7.13; no longer D6.14, D8.13
- net GS_G: now also D6.14, D7.12; no longer D7.14, D8.12
- net MISO: now also D4.15; no longer D5.15
- net MOSI: now also D4.14, D9.2; no longer D12.2, D5.14
- net N$1: now also D8.4, H3.4; no longer D9.4, H11.4
- net N$33: now also R22.1; no longer R17.1
- net N$35: now also R23.1; no longer R18.1
- net N$36: now also R28.1; no longer R23.1
- net N$37: now also R27.1; no longer R22.1
- net N$38: now also D9.5; no longer D12.5
- net N$39: now also D9.6; no longer D12.6
- net N$40: now also D9.7; no longer D12.7
- net N$41: now also D9.8; no longer D12.8
- net N$42: now also D9.9; no longer D12.9
- net N$43: now also D9.10; no longer D12.10
- net N$44: now also D9.11; no longer D12.11
- net N$45: now also D9.12; no longer D12.12
- net N$46: now also D9.13; no longer D12.13
- net N$47: now also D9.14; no longer D12.14
- net N$48: now also D9.15; no longer D12.15
- net N$49: now also D9.16; no longer D12.16
- net N$50: now also D9.17; no longer D12.17
- net N$51: now also D9.18; no longer D12.18
- net N$52: now also D9.19; no longer D12.19
- net N$53: now also D9.20; no longer D12.20
- net N$54: now also D9.23, R32.2; no longer D12.23, R30.2
- net N$56: now also R25.1; no longer R20.1
- net N$58: now also R9.2; no longer R6.2
- net N$7: now also R21.1; no longer R16.1
- net N$78: now also R26.1; no longer R21.1
- net N$80: now also R24.1; no longer R19.1
- net N$9: now also R10.2; no longer R7.2
- net PAUSE_CNT: now also S14.4; no longer S13.4
- net PL_DIN: now also D8.2; no longer D9.2
- net PS0: now also D7.3; no longer D8.3
- net PS1: now also D7.6; no longer D8.6
- net PS2: now also D7.8; no longer D8.8
- net PS3: now also D5.15, D6.5; no longer D6.15, D7.5
- net PSGS: now also D7.11; no longer D8.11
- net PS_B0: now also D5.9, D7.1; no longer D6.9, D8.1
- net PS_B1: now also D5.7, D7.4; no longer D6.7, D8.4
- net PS_B2: now also D5.6, D7.10; no longer D6.6, D8.10
- net PS_G0: now also D6.9, D7.2; no longer D7.9, D8.2
- net PS_G1: now also D6.7, D7.5; no longer D7.7, D8.5
- net PS_G2: now also D6.6, D7.9; no longer D7.6, D8.9
- net Q0_SW_BD: now also D5.3, R12.1; no longer D6.3, R28.1
- net Q0_SW_GD: now also D6.3, R17.1; no longer D7.3, R35.1
- net Q1_SW_BD: now also D5.2, R13.1; no longer D6.2, R31.1
- net Q1_SW_GD: now also D6.2, R18.1; no longer D7.2, R36.1
- net Q2_SW_BD: now also D5.1, R14.1; no longer D6.1, R32.1
- net Q2_SW_GD: now also D6.1, R19.1; no longer D7.1, R37.1
- net Q3_SW_BD: now also D5.13, R15.1; no longer D6.13, R33.1
- net Q3_SW_GD: now also D6.13, R20.1; no longer D7.13, R38.1
- net RESET_CNT: now also S15.3; no longer S14.3
- net RKR: now also S12.3; no longer S11.3
- net SCK: now also D4.16, D9.3; no longer D12.3, D5.16
- net SRC_SW_BD: now also D5.4, R11.1; no longer D6.4, R27.1
- net SRC_SW_GD: now also D6.4, R16.1; no longer D7.4, R34.1
- net STP_CS: now also D9.4; no longer D12.4, R29.2
- net VREF: now also C5.1, D4.2, R1.1, R6.1, R7.1; no longer C4.1, D5.2, R10.1, R11.1, R9.1
Routing:
- net +3V3: track 719.2 -> 673.7 mm, vias 6 -> 5
- net GND: track 24.0 -> 35.4 mm
- net ADC088S052_!CS: track 80.5 -> 72.3 mm
- net 23S08_!CS: track 56.8 -> 50.7 mm
- net N$2 (its old number): track 5.87 -> 0.00 mm
- net N$4: track 0.00 -> 5.57 mm
- net EC11_SW: track 65.1 -> 62.2 mm
- net EC11_B: track 78.1 -> 75.2 mm
- net EC11_A: track 79.4 -> 76.5 mm
