File: eagle/hwep_sequencer_v2/Beilage.sch (EAGLE design)
At the start: 127 parts, among them X1 ESP32CLIP2122

Commit message: Finalised Board
Parts:
- R27, R28, R31, R32, R33, R34, R35, R36, R37, R38: value 18k -> 47k
Other:
- note added: "Prescaler Switches Pullup Resisors"
- moved on the sheet: R27, R28, R31, R32, R33, R34, R35, R36, R37, R38

Commit message: finale gerber generation
Parts:
- removed C28: 1u, rcl_GruS:C-EUC0805
- removed C30: 100n, rcl_GruS:C-EUC0805
- removed D12: STP16CP05TTR, ic_GruS:STP16CP05TTR
- removed R33, R34, R35, R36, R37, R38: 47k, rcl_GruS:R-EUSR0805
- added C2: 1u, rcl_GruS:C-EUC0805
- added C25: 100n, rcl_GruS:C-EUC0805
- added D4: ADC088S052, adc-dac_GruS:ADC088S052
- C10: value 1u -> 100n
- C23, C8: value 100n -> 1u
- C3: value 1u -> 10n
- C4: value 4u7 -> 10n
- C5, C6: value 10n -> 100n
- C7: value 100n -> 4u7
- D5: value ADC088S052 -> 74HC148N; device adc-dac_GruS:ADC088S052 -> 74xx_GruS:74HC148N; CATEGORY 2 -> 13
- D7: value 74HC148N -> 74HC00N; device 74xx_GruS:74HC148N -> 74xx_GruS:74HC00N
- D8: value 74HC00N -> 74AHC1G125DBV; device 74xx_GruS:74HC00N -> 74xx_GruS:74AHC1G125DBV
- D9: value 74AHC1G125DBV -> STP16CP05TTR; device 74xx_GruS:74AHC1G125DBV -> ic_GruS:STP16CP05TTR
- R1: device rcl_GruS:R-EUSR0805 -> rcl_GruS:P160LB
- R10, R9: value 10k -> 1k; device rcl_GruS:P160LB -> rcl_GruS:R-EUSR0805
- R11: value 10k -> 47k; device rcl_GruS:P160LB -> rcl_GruS:R-EUSR0805
- R12, R13, R14, R15: value 10k -> 47k
- R16, R17, R18, R19, R20: value 100R -> 47k; device rcl_GruS:R-EU_R0805 -> rcl_GruS:R-EUSR0805
- R24, R25, R26: value 100k -> 100R; device rcl_GruS:R-EUSR0805 -> rcl_GruS:R-EU_R0805
- R27, R28: value 47k -> 100R; device rcl_GruS:R-EUSR0805 -> rcl_GruS:R-EU_R0805
- R29: value 10k -> 100k
- R30: value 2k7 -> 100k
- R31: value 47k -> 100k
- R32: value 47k -> 2k7
- R6, R7: value 1k -> 10k; device rcl_GruS:R-EUSR0805 -> rcl_GruS:P160LB
- S11: value (none) -> EC11E09244AQ; device switch_GruS:TASTE10XX -> switch_GruS:EC11E09244AQ
- S15: value EC11E09244AQ -> (none); device switch_GruS:EC11E09244AQ -> switch_GruS:TASTE10XX
- renumbered C29 to C24, H34 to H18, H35 to H19, H36 to H20, H37 to H21, H38 to H22, H39 to H23, H40 to H24, H41 to H25, H42 to H26, H43 to H27, H44 to H28, H45 to H29, H46 to H30, H47 to H31, H48 to H32, H49 to H33
Connections:
- removed net N$2 (its old number): H14.DO, H3.DI
- new net N$4: H11.DI, H8.DO
- net +3V3: now also C2.1, C23.1, C25.1, C6.1, D4.VD, D5.0, D5.1, D5.2, D5.VCC, D7P.VCC, D9.VDD, R11.2, R16.2, R17.2, R18.2, R19.2, R20.2; no longer C10.1, C28.1, C3.1, C30.1, D12.VDD, D5.VD, D7.0, D7.1, D7.2, D7.VCC, D8P.VCC, R1.2, R27.2, R28.2, R31.2, R32.2, R33.2, R34.2, R35.2, R36.2, R37.2, R38.2
- net +5V: now also C10.1, D8P.VCC; no longer C23.1, D9P.VCC
- net 23S08_!CS: no longer R1.1
- net 7SEG_A: now also R28.2; no longer R23.2
- net 7SEG_B: now also R27.2; no longer R22.2
- net 7SEG_C: now also R26.2; no longer R21.2
- net 7SEG_CE: now also R29.2; no longer R24.2
- net 7SEG_CH: now also R31.2; no longer R26.2
- net 7SEG_CZ: now also R30.2; no longer R25.2
- net 7SEG_D: now also R25.2; no longer R20.2
- net 7SEG_DP: now also R21.2; no longer R16.2
- net 7SEG_E: now also R24.2; no longer R19.2
- net 7SEG_F: now also R23.2; no longer R18.2
- net 7SEG_G: now also R22.2; no longer R17.2
- net ADC0: now also D4.IN0, R1.3; no longer D5.IN0, R8.3
- net ADC088S052_!CS: now also D4.!CS; no longer D5.!CS, R15.1
- net ADC1: now also D4.IN1, R2.3; no longer D5.IN1, R9.3
- net ADC2: now also D4.IN2, R3.3; no longer D5.IN2, R10.3
- net ADC3: now also D4.IN3, R4.3; no longer D5.IN3, R11.3
- net ADC4: now also D4.IN4, R5.3; no longer D5.IN4, R2.3
- net ADC5: now also D4.IN5, R6.3; no longer D5.IN5, R3.3
- net ADC6: now also D4.IN6, R7.3; no longer D5.IN6, R4.3
- net ADC7: now also D4.IN7, R8.3; no longer D5.IN7, R5.3
- net AGND: now also C5.2, D4.AGND, R1.2, R6.2, R7.2; no longer C4.2, D5.AGND, R10.2, R11.2, R9.2
- net EC11_A: now also C3.1, S11.CW; no longer C5.1, R12.1, S15.CW
- net EC11_B: now also C4.1, S11.CCW; no longer C6.1, R13.1, S15.CCW
- net EC11_SW: now also S11.NO; no longer R14.1, S15.NO
- net EVENT: now also S13.S; no longer S12.S
- net GND: now also C2.2, C25.2, C4.2, D4.DGND, D5.EI, D5.GND, D7P.GND, D8G$1.!OE, D9.!OE!/!DM2, D9.GND, R10.1, R31.1, R32.1, R9.1, S11.COM, S11.MH1, S11.MH2, S11.WIPER, S15.P, S15.P1; no longer C28.2, C30.2, C5.2, D12.!OE!/!DM2, D12.GND, D5.DGND, D6.EI, D7.GND, D9G$1.!OE, D9P.GND, R24.1, R25.1, R26.1, R6.1, R7.1, S11.P, S11.P1, S15.COM, S15.MH1, S15.MH2, S15.WIPER
- net GS_B: now also D5.GS, D7D.A; no longer D6.GS, D8D.A
- net GS_G: now also D6.GS, D7D.B; no longer D7.GS, D8D.B
- net MISO: now also D4.DOUT; no longer D5.DOUT
- net MOSI: now also D4.DIN, D9.SDI; no longer D12.SDI, D5.DIN
- net N$1: now also D8G$1.Y, H3.DI; no longer D9G$1.Y, H11.DI
- net N$33: now also R22.1; no longer R17.1
- net N$35: now also R23.1; no longer R18.1
- net N$36: now also R28.1; no longer R23.1
- net N$37: now also R27.1; no longer R22.1
- net N$38: now also D9.!OUT0; no longer D12.!OUT0
- net N$39: now also D9.!OUT1; no longer D12.!OUT1
- net N$40: now also D9.!OUT2; no longer D12.!OUT2
- net N$41: now also D9.!OUT3; no longer D12.!OUT3
- net N$42: now also D9.!OUT4; no longer D12.!OUT4
- net N$43: now also D9.!OUT5; no longer D12.!OUT5
- net N$44: now also D9.!OUT6; no longer D12.!OUT6
- net N$45: now also D9.!OUT7; no longer D12.!OUT7
- net N$46: now also D9.!OUT8; no longer D12.!OUT8
- net N$47: now also D9.!OUT9; no longer D12.!OUT9
- net N$48: now also D9.!OUT10; no longer D12.!OUT10
- net N$49: now also D9.!OUT11; no longer D12.!OUT11
- net N$50: now also D9.!OUT12; no longer D12.!OUT12
- net N$51: now also D9.!OUT13; no longer D12.!OUT13
- net N$52: now also D9.!OUT14; no longer D12.!OUT14
- net N$53: now also D9.!OUT15; no longer D12.!OUT15
- net N$54: now also D9.R-EXT, R32.2; no longer D12.R-EXT, R30.2
- net N$56: now also R25.1; no longer R20.1
- net N$58: now also R9.2; no longer R6.2
- net N$7: now also R21.1; no longer R16.1
- net N$78: now also R26.1; no longer R21.1
- net N$80: now also R24.1; no longer R19.1
- net N$9: now also R10.2; no longer R7.2
- net PAUSE_CNT: now also S14.S1; no longer S13.S1
- net PL_DIN: now also D8G$1.A; no longer D9G$1.A
- net PS0: now also D7A.Y; no longer D8A.Y
- net PS1: now also D7B.Y; no longer D8B.Y
- net PS2: now also D7C.Y; no longer D8C.Y
- net PS3: now also D5.EO, D6.EI; no longer D6.EO, D7.EI
- net PSGS: now also D7D.Y; no longer D8D.Y
- net PS_B0: now also D5.A0, D7A.A; no longer D6.A0, D8A.A
- net PS_B1: now also D5.A1, D7B.A; no longer D6.A1, D8B.A
- net PS_B2: now also D5.A2, D7C.A; no longer D6.A2, D8C.A
- net PS_G0: now also D6.A0, D7A.B; no longer D7.A0, D8A.B
- net PS_G1: now also D6.A1, D7B.B; no longer D7.A1, D8B.B
- net PS_G2: now also D6.A2, D7C.B; no longer D7.A2, D8C.B
- net Q0_SW_BD: now also D5.6, R12.1; no longer D6.6, R28.1
- net Q0_SW_GD: now also D6.6, R17.1; no longer D7.6, R35.1
- net Q1_SW_BD: now also D5.5, R13.1; no longer D6.5, R31.1
- net Q1_SW_GD: now also D6.5, R18.1; no longer D7.5, R36.1
- net Q2_SW_BD: now also D5.4, R14.1; no longer D6.4, R32.1
- net Q2_SW_GD: now also D6.4, R19.1; no longer D7.4, R37.1
- net Q3_SW_BD: now also D5.3, R15.1; no longer D6.3, R33.1
- net Q3_SW_GD: now also D6.3, R20.1; no longer D7.3, R38.1
- net RESET_CNT: now also S15.S; no longer S14.S
- net RKR: now also S12.S; no longer S11.S
- net SCK: now also D4.SCLK, D9.CLK; no longer D12.CLK, D5.SCLK
- net SRC_SW_BD: now also D5.7, R11.1; no longer D6.7, R27.1
- net SRC_SW_GD: now also D6.7, R16.1; no longer D7.7, R34.1
- net STP_CS: now also D9.LE/DM1; no longer D12.LE/DM1, R29.2
- net VREF: now also C5.1, D4.VA, R1.1, R6.1, R7.1; no longer C4.1, D5.VA, R10.1, R11.1, R9.1
